Commit message: Add moveit config and endeffector links for fingertip

File: human_arm_description/model/human_arm.urdf.xacro (robot description, xacro)
@@ -47,4 +47,15 @@
 		</link>
 	</xacro:macro>
+	<!-- end effector -->
+	<xacro:macro name="endeffector"
+	             params="link_prefix:=^|'' joint_prefix:=^|''
+	                     finger:=^ joint link parent reflect:=^ *origin">
+		<joint name="${joint_prefix}${finger}_${joint}_joint" type="fixed">
+			<xacro:insert_block name="origin"/>
+			<parent link="${link_prefix}${parent}"/>
+			<child link="${link_prefix}${finger}_${link}_link"/>
+		</joint>
+		<link name="${link_prefix}${finger}_${link}_link"/>
+	</xacro:macro>
 	<!-- FINGER MODEL -->
 	<xacro:macro name="finger"
@@ -53,4 +64,5 @@
 		<xacro:property name="proximal_len" value="${properties['link_lengths'][finger]['proximal']}"/>
 		<xacro:property name="middle_len" value="${properties['link_lengths'][finger]['middle']}"/>
+		<xacro:property name="distal_len" value="${properties['link_lengths'][finger]['distal']}"/>
 		<!-- KNUCKLE -->
 		<xacro:segment joint="abduction" link="knuckle" parent="${parent}" mesh="0">
@@ -73,4 +85,8 @@
 			<axis xyz="1 0 0" />
 		</xacro:segment>
+		<!-- TIP-->
+		<xacro:endeffector joint="ee" link="ee" parent="${finger}_distal_link">
+			<origin xyz="0 0 ${distal_len*scale_factor}" rpy="0 0 0"/>
+		</xacro:endeffector>
 	</xacro:macro>
 	<!-- THUMB MODEL -->
@@ -80,4 +96,5 @@
 		<xacro:property name="proximal_len" value="${properties['link_lengths'][finger]['proximal']}"/>
 		<xacro:property name="middle_len" value="${properties['link_lengths'][finger]['middle']}"/>
+		<xacro:property name="distal_len" value="${properties['link_lengths'][finger]['distal']}"/>
 		<!-- KNUCKLE -->
 		<xacro:segment joint="abduction" link="knuckle" parent="${parent}"
@@ -101,4 +118,8 @@
 			<axis xyz="0 ${-1*reflect} 0" />
 		</xacro:segment>
+		<!-- TIP-->
+		<xacro:endeffector joint="ee" link="ee" parent="${finger}_distal_link">
+			<origin xyz="0 0 ${distal_len*scale_factor}" rpy="0 0 0"/>
+		</xacro:endeffector>
 	</xacro:macro>
 	<!-- HUMAN HAND MODEL -->

Commit message: Add dexmo_ref link

File: human_arm_description/model/human_arm.urdf.xacro (robot description, xacro)
@@ -226,4 +226,11 @@
 			<origin xyz="${-0.04175*reflect*scale_factor} ${-0.003*scale_factor} ${0.079*scale_factor}" rpy="0 0 0"/>
 		</xacro:finger>
+		<!-- Dexmo Ref -->
+		<link name="dexmo_ref"/>
+		<joint name="${joint_prefix}dexmo_ref_static" type="fixed">
+			<parent link="middle_knuckle_link" />
+			<child link="dexmo_ref"/>
+			<origin xyz="0 0.03 -${properties['link_lengths']['dexmo_ref']}" rpy="0 0 0"/>
+		</joint>
 	</xacro:macro>
 </robot>

Commit message: Adds possibility to override link_lenghts
Link lenghts are now also used to scale MCP origins with respect to the
palm_link

File: human_arm_description/model/human_arm.urdf.xacro (robot description, xacro)
@@ -62,7 +62,7 @@
 	             params="parent link_prefix:=^|'' joint_prefix:=^|''
 	                     finger reflect:=^ *origin joint_props:=${properties['joints']}">
-		<xacro:property name="proximal_len" value="${properties['link_lengths'][finger]['proximal']}"/>
-		<xacro:property name="middle_len" value="${properties['link_lengths'][finger]['middle']}"/>
-		<xacro:property name="distal_len" value="${properties['link_lengths'][finger]['distal']}"/>
+		<xacro:property name="proximal_len" value="${link_lengths[finger]['proximal']}"/>
+		<xacro:property name="middle_len" value="${link_lengths[finger]['middle']}"/>
+		<xacro:property name="distal_len" value="${link_lengths[finger]['distal']}"/>
 		<!-- KNUCKLE -->
 		<xacro:segment joint="abduction" link="knuckle" parent="${parent}" mesh="0">
@@ -94,7 +94,7 @@
 	             params="parent link_prefix:=^|'' joint_prefix:=^|''
 	                     finger:='thumb' reflect:=^ *origin joint_props:=${properties['joints']}">
-		<xacro:property name="proximal_len" value="${properties['link_lengths'][finger]['proximal']}"/>
-		<xacro:property name="middle_len" value="${properties['link_lengths'][finger]['middle']}"/>
-		<xacro:property name="distal_len" value="${properties['link_lengths'][finger]['distal']}"/>
+		<xacro:property name="proximal_len" value="${link_lengths[finger]['proximal']}"/>
+		<xacro:property name="middle_len" value="${link_lengths[finger]['middle']}"/>
+		<xacro:property name="distal_len" value="${link_lengths[finger]['distal']}"/>
 		<!-- KNUCKLE -->
 		<xacro:segment joint="abduction" link="knuckle" parent="${parent}"
@@ -126,8 +126,14 @@
 	<xacro:macro name="human_arm"
 	             params="parent link_prefix:=^|'' joint_prefix:=^|'' scale:=1.0
-	                     use_synergy side:='' *origin">
+	                     use_synergy side:='' link_length_override=^|'' *origin">
 		<!-- load kinematics properties -->
 		<xacro:property name="package" value="$(find human_arm_description)"/>
-		<xacro:property name="properties" value="${load_yaml(package + '/model/properties.yaml')}"/>
+		<xacro:property name="properties" value="${xacro.load_yaml(package + '/model/properties.yaml')}"/>
+		<xacro:if value="${ link_length_override == '' }" >
+			<xacro:property name="link_lengths" value="${properties['link_lengths']}"/>
+		</xacro:if>
+		<xacro:unless value="${ link_length_override == '' }" >
+			<xacro:property name="link_lengths" value="${xacro.load_yaml(link_length_override)}"/>
+		</xacro:unless>
 		<xacro:property name="synergies" value="${properties['synergies']}"/>
 		<xacro:property name="scale_factor" value="${scale}"/>
@@ -155,6 +161,6 @@
 		<!-- WRIST (Supination/Pronation) -->
 		<joint name="${joint_prefix}distal_radioulnar_joint" type="revolute" >
-			<xacro:property name="forearm_y" value="${properties['link_lengths']['forearm']['y']}"/>
-			<xacro:property name="forearm_z" value="${properties['link_lengths']['forearm']['z']}"/>
+			<xacro:property name="forearm_y" value="${link_lengths['forearm']['y']}"/>
+			<xacro:property name="forearm_z" value="${link_lengths['forearm']['z']}"/>
 			<origin xyz="0 ${scale_factor*forearm_y} ${scale_factor*forearm_z}" rpy="0 0 0" />
 			<axis xyz="0 0 ${-1*reflect}" />
@@ -212,17 +218,17 @@
 		<!-- THUMB AND FINGERS -->
 		<xacro:thumb parent="palm_link" finger="thumb">
-			<origin xyz="${0.02475*reflect*scale_factor} ${-0.0125*scale_factor} ${0.0125*scale_factor}" rpy="0.0 ${0.6240*reflect} 0"/>
+			<origin xyz="${link_lengths['palm_link_distances']['thumb']['x']*reflect*scale_factor} ${link_lengths['palm_link_distances']['thumb']['y']*scale_factor} ${link_lengths['palm_link_distances']['thumb']['z']*scale_factor}" rpy="0.0 ${0.6240*reflect} 0"/>
 		</xacro:thumb>
 		<xacro:finger parent="palm_link" finger="index">
-			<origin xyz="${0.02175*reflect*scale_factor} ${-0.002*scale_factor} ${0.099*scale_factor}" rpy="0 0 0"/>
+			<origin xyz="${link_lengths['palm_link_distances']['index']['x']*reflect*scale_factor} ${link_lengths['palm_link_distances']['index']['y']*scale_factor} ${link_lengths['palm_link_distances']['index']['z']*scale_factor}" rpy="0 0 0"/>
 		</xacro:finger>
 		<xacro:finger parent="palm_link" finger="middle">
-			<origin xyz="${-0.002*reflect*scale_factor} ${0.0015*scale_factor} ${0.0955*scale_factor}" rpy="0 0 0"/>
+			<origin xyz="${link_lengths['palm_link_distances']['middle']['x']*reflect*scale_factor} ${link_lengths['palm_link_distances']['middle']['y']*scale_factor} ${link_lengths['palm_link_distances']['middle']['z']*scale_factor}" rpy="0 0 0"/>
 		</xacro:finger>
 		<xacro:finger parent="palm_link" finger="ring">
-			<origin xyz="${-0.02225*reflect*scale_factor} ${0.0010*scale_factor} ${0.090*scale_factor}" rpy="0 0 0"/>
+			<origin xyz="${link_lengths['palm_link_distances']['ring']['x']*reflect*scale_factor} ${link_lengths['palm_link_distances']['ring']['y']*scale_factor} ${link_lengths['palm_link_distances']['ring']['z']*scale_factor}" rpy="0 0 0"/>
 		</xacro:finger>
 		<xacro:finger parent="palm_link" finger="little">
-			<origin xyz="${-0.04175*reflect*scale_factor} ${-0.003*scale_factor} ${0.079*scale_factor}" rpy="0 0 0"/>
+			<origin xyz="${link_lengths['palm_link_distances']['little']['x']*reflect*scale_factor} ${link_lengths['palm_link_distances']['little']['y']*scale_factor} ${link_lengths['palm_link_distances']['little']['z']*scale_factor}" rpy="0 0 0"/>
 		</xacro:finger>
 		<!-- Dexmo Ref -->
@@ -231,5 +237,5 @@
 			<parent link="middle_knuckle_link" />
 			<child link="dexmo_ref"/>
-			<origin xyz="0 0.03 -${properties['link_lengths']['dexmo_ref']}" rpy="0 0 0"/>
+			<origin xyz="0 0.03 -${link_lengths['dexmo_ref']}" rpy="0 0 0"/>
 		</joint>
 	</xacro:macro>

File: human_arm_description/robots/human_arm.urdf.xacro (robot description, xacro)
@@ -10,4 +10,5 @@
 	<xacro:arg name="side" default="right"/>
 	<xacro:arg name="use_synergy" default="false"/>
+	<xacro:arg name="link_length_override" default="" />
 	<xacro:include filename="../model/human_arm.urdf.xacro"/>
 	<link name="$(arg prefix)forearm_base"/>
@@ -16,4 +17,5 @@
 	                  link_prefix="$(arg link_prefix)" joint_prefix="$(arg joint_prefix)"
 	                  scale="$(arg scale)"
+					  link_length_override="$(arg link_length_override)"
 			  side="$(arg side)" use_synergy="$(arg use_synergy)">
 		<origin xyz="0 0 0" rpy="0 0 0"/>

Commit message: Fix dexmo_ref position

File: human_arm_description/model/human_arm.urdf.xacro (robot description, xacro)
@@ -237,5 +237,5 @@
 			<parent link="middle_knuckle_link" />
 			<child link="dexmo_ref"/>
-			<origin xyz="0 0.03 -${link_lengths['dexmo_ref']}" rpy="0 0 0"/>
+			<origin xyz="0 0.012 -${link_lengths['dexmo_ref']}" rpy="0 0 0"/>
 		</joint>
 	</xacro:macro>

Commit message: Fix default finger tip positions

File: human_arm_description/model/human_arm.urdf.xacro (robot description, xacro)
@@ -87,5 +87,5 @@
 		<!-- TIP-->
 		<xacro:endeffector joint="ee" link="ee" parent="${finger}_distal_link">
-			<origin xyz="0 0 ${distal_len*scale_factor}" rpy="0 0 0"/>
+			<origin xyz="0 0.0027 ${distal_len*scale_factor}" rpy="0 0 0"/>
 		</xacro:endeffector>
 	</xacro:macro>
@@ -120,5 +120,5 @@
 		<!-- TIP-->
 		<xacro:endeffector joint="ee" link="ee" parent="${finger}_distal_link">
-			<origin xyz="0 0 ${distal_len*scale_factor}" rpy="0 0 0"/>
+			<origin xyz="0.005 0 ${distal_len*scale_factor}" rpy="0 0 0"/>
 		</xacro:endeffector>
 	</xacro:macro>

Commit message: Switch dexmo_ref parent to palm_link

File: human_arm_description/model/human_arm.urdf.xacro (robot description, xacro)
@@ -235,7 +235,7 @@
 		<link name="dexmo_ref"/>
 		<joint name="${joint_prefix}dexmo_ref_static" type="fixed">
-			<parent link="middle_knuckle_link" />
+			<parent link="palm_link" />
 			<child link="dexmo_ref"/>
-			<origin xyz="0 0.012 -${link_lengths['dexmo_ref']}" rpy="0 0 0"/>
+			<origin xyz="${link_lengths['palm_link_distances']['middle']['x']} 0.0135 ${link_lengths['palm_link_distances']['middle']['z'] - link_lengths['dexmo_ref']}" rpy="0 0 0"/>
 		</joint>
 	</xacro:macro>
